File: freq.kicad_pcb (KiCad board)
At the start: 2 copper layers, 63.5 x 45 mm, 69 parts, among them J2 Screw_Terminal_01x02, J3 Conn_01x03, J4 Conn_01x04, J5 Screw_Terminal_01x03, J6 Conn_01x04, Q1 Q_NMOS_GDS, Q2 Q_NMOS_GDS, Q3 Q_NMOS_GDS, Q4 Q_NMOS_GDS, Q5 Q_NMOS_GDS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

Commit message: update kicad version
Other:
- net class Default removed
